File: HW/kicad/Z79Forth.sch (KiCad schematic (older format))
At the start: 24 parts, among them J1 HX-2118P, Q1 BS170, U1 74HCT74, U10 AT28C64B-15PU, U11 F84256-10LL, U12 74HCT245, U2 74HCT112E, U3 74HC14, U4 74HCT00, U5 74HCT138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

Commit message: Update schematics to version 2.2.1.
Parts:
- RN2: value 10K x 5 -> 1K x 5
- renumbered R5 to R3
Changed lines of the file:
@@
 Sheet 1 2
 Title "Z79Forth Reference Board"
-Date "2021-10-28"
-Rev "2.2"
+Date "2022-01-26"
+Rev "2.2.1"
 Comp "Francois Laagel"
 Comment1 " "
@@
 Text GLabel 7050 5750 0    39   Input ~ 0
 ~DEV0
-Text GLabel 7050 4750 0    50   Input ~ 0
+Text GLabel 7050 4750 0    50   BiDi ~ 0
 D0
-Text GLabel 7050 4850 0    50   Input ~ 0
+Text GLabel 7050 4850 0    50   BiDi ~ 0
 D1
-Text GLabel 7050 4950 0    50   Input ~ 0
+Text GLabel 7050 4950 0    50   BiDi ~ 0
 D2
-Text GLabel 7050 5050 0    50   Input ~ 0
+Text GLabel 7050 5050 0    50   BiDi ~ 0
 D3
-Text GLabel 7050 5150 0    50   Input ~ 0
+Text GLabel 7050 5150 0    50   BiDi ~ 0
 D4
-Text GLabel 7050 5250 0    50   Input ~ 0
+Text GLabel 7050 5250 0    50   BiDi ~ 0
 D5
-Text GLabel 7050 5350 0    50   Input ~ 0
+Text GLabel 7050 5350 0    50   BiDi ~ 0
 D6
-Text GLabel 7050 5450 0    50   Input ~ 0
+Text GLabel 7050 5450 0    50   BiDi ~ 0
 D7
 Wire Wire Line
@@
 P 4600 1550
 F 0 "RN2" H 4888 1596 50  0000 L CNN
-F 1 "10K x 5" H 4888 1505 50  0000 L CNN
+F 1 "1K x 5" H 4888 1505 50  0000 L CNN
 F 2 "Resistor_THT:R_Array_SIP6" V 4975 1550 50  0001 C CNN
 F 3 "http://www.vishay.com/docs/31509/csc.pdf" H 4600 1550 50  0001 C CNN
@@
 	4250 6850 3700 6850
 $Comp
-L Device:R R5
+L Device:R R3
 U 1 1 61882744
 P 4250 6700
-F 0 "R5" V 4150 6700 50  0000 C CNN
+F 0 "R3" V 4150 6700 50  0000 C CNN
 F 1 "10K" V 4250 6700 50  0000 C CNN
 F 2 "" V 4180 6700 50  0001 C CNN
