File: HW/kicad/file615D6455.sch (KiCad schematic (older format))
At the start: 22 parts, among them J2 FT232RL-Breakout, J3 IDC10-Male, J4 IDC50-Male, U13 Max232IN, U3 74HCT14, U6 74HCT02, U9 HD63B50

Commit message: Update schematics to version 2.2.1.
Parts:
- removed R3: 10K, symbol Device:R
- added C11: 1 uF, symbol Device:C
- added C12: 10000 uF, symbol Device:C_Polarized
- added R5: 100K, symbol Device:R
- added S2: DPST-NO, symbol Switch:SW_DPST
- added U14: ATF22V10C-7PX, symbol Z79Forth:ATF22V10C-7PX
- added U15: MC146818P, Package_DIP:DIP-40_W15.24mm, symbol Z79Forth:MC146818P
- added Y3: DS32kHz-N, Oscillator:Oscillator_DIP-14, symbol Z79Forth:DS32kHz-N
- R4: value 10K -> 47K
- U13: value Max232IN -> Max232EPE+
- U3: value 74HCT14 -> 74HC14
Connections:
- net A0: now also U14.9 (I7)
- net D0: now also U15.4 (AD0)
- net D1: now also U15.5 (AD1)
- net D2: now also U15.6 (AD2)
- net D3: now also U15.7 (AD3)
- net D4: now also U15.8 (AD4)
- net D5: now also U15.9 (AD5)
- net D6: now also U15.10 (AD6)
- net D7: now also U15.11 (AD7)
- net E: now also U14.4 (I2)
- net GND: now also C11.2, C12.2, R5.2, U14.12 (GND), U15.12 (VSS), U15.13 (CE), Y3.4 (GND); no longer U3.3
- net SYSCLK: now also U14.1 (CLK)
- net VCC: now also C12.1, U14.24 (VCC), U15.20 (CKFS), U15.22 (PS), U15.24 (VDD), Y3.13 (Vcc)
- net ~CFRST: now also U14.2 (I0), U15.18 (~RESET)
- net ~DEV5: now also U14.5 (I3), U14.8 (I6)
- net ~FIRQ: now also U15.19 (~IRQ)
- net ~NMI: now also U3.4
- net ~Q: now also U14.3 (I1)
- net ~RRTS: no longer R4.2
- net ~STRETCH: now also U14.14 (O9)
- net ~WR: now also U14.7 (I5), U15.15 (R/~W)
- new net: C11.1, R5.1, S2.2, S2.4, U3.3
- new net: U14.21 (O2), U15.14 (AS)
- new net: U14.20 (O3), U15.17 (DS)
- new net: U15.2 (OSC1), Y3.12 (32kHz)
- new net: R4.2, S2.1, S2.3
- no-connect marks 17 -> 31
Other:
- note added: "Experimental--not a part of the reference design"
- moved on the sheet: J4, U3B, U6B, U6C, U6D
